File: RFB/RFB.kicad_sch (KiCad schematic)
At the start: 55 parts, among them IC1 SKY67189-396LF, J1 Conn_Coaxial, J10 Conn_02x06_Odd_Even, J2 Conn_Coaxial, J3 Conn_Coaxial, J4 Conn_01x16_MountingPin, J5 Conn_01x04, J6 Conn_01x03_Male, J9 Conn_01x02_Male, U1 TG2016SMN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

Commit message: 2
Parts:
- J7: value (none) -> Conn_02x06_Odd_Even; footprint (none) -> Connector_PinSocket_2.54mm:PinSocket_2x06_P2.54mm_Vertical
- J8: value (none) -> Conn_01x01; footprint (none) -> Connector_PinSocket_2.54mm:PinSocket_1x01_P2.54mm_Vertical
- SW1: value (none) -> PH3; footprint (none) -> Button_Switch_SMD:SW_SPST_PTS810
- SW2: value (none) -> RST; footprint (none) -> Button_Switch_SMD:SW_SPST_PTS810
Changed lines of the file:
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@@
       (effects (font (size 1.27 1.27)) (justify left))
     )
-    (property "Value" "" (id 1) (at 200.152 127.4322 0)
-      (effects (font (size 1.27 1.27)) (justify left))
-    )
-    (property "Footprint" "" (id 2) (at 198.12 125.73 0)
+    (property "Value" "Conn_01x01" (id 1) (at 200.152 127.4322 0)
+      (effects (font (size 1.27 1.27)) (justify left))
+    )
+    (property "Footprint" "Connector_PinSocket_2.54mm:PinSocket_1x01_P2.54mm_Vertical" (id 2) (at 198.12 125.73 0)
       (effects (font (size 1.27 1.27)) hide)
     )
@@
     (in_bom yes) (on_board yes)
     (property "Reference" "J7" (id 0) (at 184.15 99.1702 0))
-    (property "Value" "" (id 1) (at 184.15 101.7071 0))
-    (property "Footprint" "" (id 2) (at 182.88 109.22 0)
+    (property "Value" "Conn_02x06_Odd_Even" (id 1) (at 184.15 101.7071 0))
+    (property "Footprint" "Connector_PinSocket_2.54mm:PinSocket_2x06_P2.54mm_Vertical" (id 2) (at 182.88 109.22 0)
       (effects (font (size 1.27 1.27)) hide)
     )
@@
     (in_bom yes) (on_board yes) (fields_autoplaced)
     (property "Reference" "SW2" (id 0) (at 210.82 75.9292 0))
-    (property "Value" "" (id 1) (at 210.82 78.4661 0))
-    (property "Footprint" "" (id 2) (at 210.82 77.47 0)
+    (property "Value" "RST" (id 1) (at 210.82 78.4661 0))
+    (property "Footprint" "Button_Switch_SMD:SW_SPST_PTS810" (id 2) (at 210.82 77.47 0)
       (effects (font (size 1.27 1.27)) hide)
     )
@@
     (in_bom yes) (on_board yes) (fields_autoplaced)
     (property "Reference" "SW1" (id 0) (at 173.99 89.8992 0))
-    (property "Value" "" (id 1) (at 173.99 92.4361 0))
-    (property "Footprint" "" (id 2) (at 173.99 91.44 0)
+    (property "Value" "PH3" (id 1) (at 173.99 92.4361 0))
+    (property "Footprint" "Button_Switch_SMD:SW_SPST_PTS810" (id 2) (at 173.99 91.44 0)
       (effects (font (size 1.27 1.27)) hide)
     )
@@
     )
     (path "/c82a81f1-0483-453a-b86c-a887aa014c5b/ecf5090e-8e85-4fb2-9564-a566cb26a230"
-      (reference "R69") (unit 1) (value "4k7 1%") (footprint "Resistor_SMD:R_0402_1005Metric")
+      (reference "R69") (unit 1) (value "3k 1%") (footprint "Resistor_SMD:R_0402_1005Metric")
     )
     (path "/c82a81f1-0483-453a-b86c-a887aa014c5b/321cb765-f9f4-4a30-8644-72304929598b"

Commit message: 0
Parts:
- U11: value STM32L431CBTx -> STM32L431CCT6
Connections:
- net CAN_R: now also U11.33 (PA12); no longer U11.32 (PA11)
- net CAN_T: now also U11.32 (PA11); no longer U11.33 (PA12)
- net GND: now also R41.1, SW1.2, U11.44 (PH3)
