File: RFB/_autosave-generator.kicad_sch (KiCad schematic)
At the start: 30 parts, among them U4 LMX2572RHAR, U5 TLV365DBVR

Commit message: 0
Parts:
- R10: value 4k7 -> DNP
Changed lines of the file:
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@@
       (effects (font (size 1.27 1.27)))
     )
-    (property "Value" "4k7" (at 266.7 65.1311 90)
+    (property "Value" "DNP" (at 266.7 65.1311 90)
       (effects (font (size 1.27 1.27)))
     )
