File: RFB/pa2.kicad_sch (KiCad schematic)
At the start: 31 parts, among them Q1 PJA3433, U10 AZ431LBNTR, U14 SE5004L, U15 LM321, U9 SN74LV1T34DCK

Commit message: 2
Parts:
- R40: value (none) -> 100; footprint (none) -> Resistor_SMD:R_0402_1005Metric
- RV1: value (none) -> B10k; footprint (none) -> Potentiometer_THT:Potentiometer_Piher_PT-6-H_Horizontal
Changed lines of the file:
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@@
     (in_bom yes) (on_board yes) (fields_autoplaced)
     (property "Reference" "R40" (id 0) (at 55.88 84.4636 90))
-    (property "Value" "" (id 1) (at 55.88 87.0005 90))
-    (property "Footprint" "" (id 2) (at 55.88 88.9 0)
+    (property "Value" "100" (id 1) (at 55.88 87.0005 90))
+    (property "Footprint" "Resistor_SMD:R_0402_1005Metric" (id 2) (at 55.88 88.9 0)
       (effects (font (size 1.27 1.27)) hide)
     )
@@
       (effects (font (size 1.27 1.27)) (justify right))
     )
-    (property "Value" "" (id 1) (at 82.0421 102.0322 0)
+    (property "Value" "B10k" (id 1) (at 82.0421 102.0322 0)
       (effects (font (size 1.27 1.27)) (justify right))
     )
-    (property "Footprint" "" (id 2) (at 83.82 100.33 0)
+    (property "Footprint" "Potentiometer_THT:Potentiometer_Piher_PT-6-H_Horizontal" (id 2) (at 83.82 100.33 0)
       (effects (font (size 1.27 1.27)) hide)
     )

Commit message: 0
Connections:
- net at Q1.3 (D), R21.1: no longer RV1.1
- net at C82.2, R21.2, R34.2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: now also RV1.1
