File: RFB/power.kicad_sch (KiCad schematic)
At the start: 43 parts, among them IC10 TPS74601PBDRVR, IC2 TPS74601PBDRVR, IC8 TPS74601PBDRVR, IC9 TPS74601PBDRVR, U16 XPR6272ITC5, U20 BD33GA3WNUX, U22 BD33GA3WNUX

Commit message: 2
Parts:
- R69: value 4k7 1% -> (none); footprint Resistor_SMD:R_0402_1005Metric -> (none)
Changed lines of the file:
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@@
       (effects (font (size 1.27 1.27)) (justify right))
     )
-    (property "Value" "4k7 1%" (id 1) (at 156.718 170.6122 0)
+    (property "Value" "" (id 1) (at 156.718 170.6122 0)
       (effects (font (size 1.27 1.27)) (justify right))
     )
-    (property "Footprint" "Resistor_SMD:R_0402_1005Metric" (id 2) (at 156.718 168.91 90)
+    (property "Footprint" "" (id 2) (at 156.718 168.91 90)
       (effects (font (size 1.27 1.27)) hide)
     )

Commit message: 0
Parts:
- R69: value (none) -> 3k 1%; footprint (none) -> Resistor_SMD:R_0402_1005Metric
