File: RFB/generator.kicad_sch (KiCad schematic)
At the start: 30 parts, among them U4 LMX2572RHAR, U5 TLV365DBVR

Commit message: qwf
Parts:
- C28, C29: value 3p R -> 1p5 R
Changed lines of the file:
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@@
       (effects (font (size 1.27 1.27)))
     )
-    (property "Value" "3p R" (at 208.2736 51.885 90)
+    (property "Value" "1p5 R" (at 208.2736 51.885 90)
       (effects (font (size 1.27 1.27)))
     )
@@
       (effects (font (size 1.27 1.27)))
     )
-    (property "Value" "3p R" (at 208.2736 46.805 90)
-      (effects (font (size 1.27 1.27)))
-    )
+    (property "Value" "1p5 R" (at 208.2736 46.805 90)
+      (effects (font (size 1.27 1.27)))
+    )
