File: RFB/mixer.kicad_sch (KiCad schematic)
At the start: 25 parts, among them U8 ADL5802

Commit message: qwf
Parts:
- C59, C60, C61, C62, C63, C64: value 3p R -> 1p5 R
Changed lines of the file:
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@@
       (effects (font (size 1.27 1.27)))
     )
-    (property "Value" "3p R" (at 73.6536 74.745 90)
+    (property "Value" "1p5 R" (at 73.6536 74.745 90)
       (effects (font (size 1.27 1.27)))
     )
@@
       (effects (font (size 1.27 1.27)))
     )
-    (property "Value" "3p R" (at 73.6663 120.465 90)
+    (property "Value" "1p5 R" (at 73.6663 120.465 90)
       (effects (font (size 1.27 1.27)))
     )
@@
       (effects (font (size 1.27 1.27)))
     )
-    (property "Value" "3p R" (at 73.6536 110.305 90)
+    (property "Value" "1p5 R" (at 73.6536 110.305 90)
       (effects (font (size 1.27 1.27)))
     )
@@
       (effects (font (size 1.27 1.27)))
     )
-    (property "Value" "3p R" (at 93.9736 92.525 90)
+    (property "Value" "1p5 R" (at 93.9736 92.525 90)
       (effects (font (size 1.27 1.27)))
     )
@@
       (effects (font (size 1.27 1.27)))
     )
-    (property "Value" "3p R" (at 73.6663 84.905 90)
+    (property "Value" "1p5 R" (at 73.6663 84.905 90)
       (effects (font (size 1.27 1.27)))
     )
@@
       (effects (font (size 1.27 1.27)))
     )
-    (property "Value" "3p R" (at 93.9863 100.145 90)
-      (effects (font (size 1.27 1.27)))
-    )
+    (property "Value" "1p5 R" (at 93.9863 100.145 90)
+      (effects (font (size 1.27 1.27)))
+    )
